File: 12.1.1 - PLC Connector/12.1.1 - PLC Connector.kicad_pcb (KiCad board)
At the start: 2 copper layers, 29.8 x 61.3 mm, 32 parts, among them J101 Conn_01x01_PAD, J102 Conn_01x01_PAD, J103 Conn_01x01_PAD, J104 Conn_01x01_PAD, J105 Conn_01x01_PAD, J106 Conn_01x01_PAD, J107 Conn_01x01_PAD, J108 Conn_01x01_PAD, J109 Conn_01x01_PAD, J110 Conn_01x01_PAD, J111 Conn_01x01_PAD, J112 Conn_01x01_PAD, J113 Conn_01x01_PAD, J114 Conn_01x01_PAD, J115 Conn_01x01_PAD, J116 Conn_01x01_PAD, J117 Conn_01x01_PAD, J118 DB128L-5.08-2P-BK-S, J119 Conn_01x01_PAD, J120 Conn_01x01_PAD, J121 Conn_01x01_PAD, J122 DB128L-5.08-2P-BK-S, J123 DB128L-5.08-2P-BK-S, J124 DB128L-5.08-2P-BK-S, J125 DB128L-5.08-2P-BK-S, J126 22292041

Commit message: 12.2.1 front silk
Other:
- board text added: "12.1.1"
- board text removed: "12.1.0"
Changed lines of the file:
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@@
     (effects (font (size 1.8288 1.8288) (thickness 0.4572) bold) (justify bottom mirror))
   )
-  (gr_text "12.1.0" (at 160.782 110.49 90) (layer "B.SilkS")
+  (gr_text "12.1.1" (at 160.782 110.49 90) (layer "B.SilkS")
     (effects (font (size 1.8288 1.8288) (thickness 0.4572) bold) (justify bottom mirror))
   )
