File: 12.X.2 - PLC Connector Combined/12.1.1.a.kicad_sch (KiCad schematic)
At the start: 30 parts, among them J201 Conn_01x01_PAD, J202 Conn_01x01_PAD, J203 Conn_01x01_PAD, J204 Conn_01x01_PAD, J205 Conn_01x01_PAD, J206 Conn_01x01_PAD, J207 Conn_01x01_PAD, J208 Conn_01x01_PAD, J209 Conn_01x01_PAD, J210 Conn_01x01_PAD, J211 Conn_01x01_PAD, J212 Conn_01x01_PAD, J213 Conn_01x01_PAD, J214 Conn_01x01_PAD, J215 Conn_01x01_PAD, J216 Conn_01x01_PAD, J217 Conn_01x01_PAD, J218 Conn_01x01_PAD, J219 Conn_01x01_PAD, J220 Conn_01x01_PAD, J221 Dorabo-DB128L_5_08_2P_BKS, J222 Dorabo-DB128L_5_08_2P_BKS, J223 Dorabo-DB128L_5_08_2P_BKS, J224 Dorabo-DB128L_5_08_2P_BKS, J225 Dorabo-DB128L_5_08_2P_BKS, J226 B04B-XASK-1

Commit message: Version 14.x.4 PMOS Design
Other:
- title: (none) -> PLC INPUTS
Changed lines of the file:
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@@
 (kicad_sch (version 20230121) (generator eeschema)
   (paper "A4")
+  (title_block
+    (title "PLC INPUTS")
+  )
   (junction (at 130.81 86.36) (diameter 0) (color 0 0 0 0)
   )
