File: 12.X.2 - PLC Connector Combined/12.2.1.a.kicad_sch (KiCad schematic)
At the start: 32 parts, among them J301 Conn_01x01_PAD, J302 Conn_01x01_PAD, J303 Conn_01x01_PAD, J304 Conn_01x01_PAD, J305 Conn_01x01_PAD, J306 Conn_01x01_PAD, J307 Conn_01x01_PAD, J308 Conn_01x01_PAD, J309 Conn_01x01_PAD, J310 Conn_01x01_PAD, J311 Conn_01x01_PAD, J312 Conn_01x01_PAD, J313 Conn_01x01_PAD, J314 Conn_01x01_PAD, J315 Conn_01x01_PAD, J316 Conn_01x01_PAD, J317 DB128L-5.08-2P-BK-S, J318 DB128L-5.08-3P-BK-S, J319 DB128L-5.08-2P-BK-S, J320 DB128L-5.08-2P-BK-S, J321 B04B-XASK-1

Commit message: Version 14.x.4 PMOS Design
Other:
- note added: "PLC RELAY SWITCH CIRCUIT"
- note added: "Q1:1"
- note added: "Q1:2"
- note added: "Q2:1"
- note added: "Q2:2"
- note added: "Q3:1"
- note added: "Q3:2"
- note added: "Q4:1"
- note added: "Q4:2"
- note added: "QX:1"
- note added: "QX:2"
- title: (none) -> PLC OUTPUTS (RELAY)
Changed lines of the file:
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@@
 (kicad_sch (version 20230121) (generator eeschema)
   (paper "A4")
+  (title_block
+    (title "PLC OUTPUTS (RELAY)")
+  )
   (junction (at 96.52 102.87) (diameter 0) (color 0 0 0 0)
   )
@@
     (stroke (width 0) (type default))
   )
+  (bus (pts (xy 144.78 168.91) (xy 144.78 171.45))
+    (stroke (width 0) (type default))
+  )
   (wire (pts (xy 247.65 153.67) (xy 247.65 91.44))
     (stroke (width 0) (type default))
@@
     (stroke (width 0) (type default))
   )
-  (wire (pts (xy 128.27 161.29) (xy 128.27 137.16))
+  (wire (pts (xy 96.52 161.29) (xy 96.52 137.16))
     (stroke (width 0) (type default))
   )
@@
     (stroke (width 0) (type default))
   )
+  (bus (pts (xy 144.78 179.07) (xy 158.75 179.07))
+    (stroke (width 0) (type default))
+  )
   (wire (pts (xy 208.28 29.21) (xy 208.28 38.1))
     (stroke (width 0) (type default))
@@
     (stroke (width 0) (type default))
   )
+  (bus (pts (xy 142.24 173.99) (xy 144.78 171.45))
+    (stroke (width 0) (type default))
+  )
   (wire (pts (xy 198.12 121.92) (xy 198.12 128.27))
     (stroke (width 0) (type default))
   )
+  (bus (pts (xy 158.75 168.91) (xy 144.78 168.91))
+    (stroke (width 0) (type default))
+  )
   (wire (pts (xy 127 29.21) (xy 127 34.29))
     (stroke (width 0) (type default))
@@
     (stroke (width 0) (type default))
   )
-  (wire (pts (xy 128.27 137.16) (xy 208.28 137.16))
+  (wire (pts (xy 83.82 161.29) (xy 96.52 161.29))
+    (stroke (width 0) (type default))
+  )
+  (bus (pts (xy 144.78 173.99) (xy 144.78 179.07))
     (stroke (width 0) (type default))
   )
@@
     (stroke (width 0) (type default))
   )
-  (wire (pts (xy 142.24 139.7) (xy 162.56 139.7))
+  (wire (pts (xy 101.6 139.7) (xy 162.56 139.7))
     (stroke (width 0) (type default))
   )
@@
     (stroke (width 0) (type default))
   )
-  (wire (pts (xy 142.24 171.45) (xy 83.82 171.45))
+  (wire (pts (xy 101.6 171.45) (xy 83.82 171.45))
     (stroke (width 0) (type default))
   )
@@
     (stroke (width 0) (type default))
   )
-  (wire (pts (xy 83.82 161.29) (xy 128.27 161.29))
-    (stroke (width 0) (type default))
-  )
   (wire (pts (xy 62.23 148.59) (xy 62.23 161.29))
     (stroke (width 0) (type default))
@@
     (stroke (width 0) (type default))
   )
-  (wire (pts (xy 142.24 139.7) (xy 142.24 171.45))
+  (wire (pts (xy 96.52 137.16) (xy 208.28 137.16))
+    (stroke (width 0) (type default))
+  )
+  (wire (pts (xy 101.6 139.7) (xy 101.6 171.45))
     (stroke (width 0) (type default))
   )
@@
     (stroke (width 0) (type default))
   )
+  (rectangle (start 121.92 162.56) (end 157.48 187.96)
+    (stroke (width 0) (type default))
+    (fill (type none))
+  )
+  (text "Q4:1" (at 22.86 162.56 0)
+    (effects (font (size 1.27 1.27)) (justify left bottom))
+  )
+  (text "Q4:2" (at 22.86 172.72 0)
+    (effects (font (size 1.27 1.27)) (justify left bottom))
+  )
+  (text "Q3:1" (at 22.86 102.87 0)
+    (effects (font (size 1.27 1.27)) (justify left bottom))
+  )
+  (text "QX:2" (at 158.75 180.34 0)
+    (effects (font (size 1.27 1.27)) (justify left bottom))
+  )
+  (text "PLC RELAY\nSWITCH\nCIRCUIT" (at 127 176.53 0)
+    (effects (font (size 1.27 1.27)) (justify left bottom))
+  )
+  (text "Q2:1" (at 22.86 67.31 0)
+    (effects (font (size 1.27 1.27)) (justify left bottom))
+  )
+  (text "Q1:2" (at 24.13 36.83 0)
+    (effects (font (size 1.27 1.27)) (justify left bottom))
+  )
+  (text "Q2:2" (at 22.86 77.47 0)
+    (effects (font (size 1.27 1.27)) (justify left bottom))
+  )
+  (text "Q3:2" (at 22.86 113.03 0)
+    (effects (font (size 1.27 1.27)) (justify left bottom))
+  )
+  (text "QX:1" (at 158.75 170.18 0)
+    (effects (font (size 1.27 1.27)) (justify left bottom))
+  )
+  (text "Q1:1" (at 24.13 26.67 0)
+    (effects (font (size 1.27 1.27)) (justify left bottom))
+  )
   (symbol (lib_id "PCB_Library:Conn_01x01_PAD") (at 40.64 171.45 0) (unit 1)
