File: 14.1.4 - PMOS - PLC Connector Combined/12.2.1.a.kicad_sch (KiCad schematic)
At the start: 69 parts, among them J301 Conn_01x01_PAD, J302 Conn_01x01_PAD, J303 Conn_01x01_PAD, J304 Conn_01x01_PAD, J305 Conn_01x01_PAD, J306 Conn_01x01_PAD, J307 Conn_01x01_PAD, J308 Conn_01x01_PAD, J309 Conn_01x01_PAD, J310 Conn_01x01_PAD, J311 Conn_01x01_PAD, J312 Conn_01x01_PAD, J313 Conn_01x01_PAD, J314 Conn_01x01_PAD, J315 Conn_01x01_PAD, J316 Conn_01x01_PAD, J317 DB128L-5.08-2P-BK-S, J318 DB128L-5.08-3P-BK-S, J319 DB128L-5.08-2P-BK-S, J320 DB128L-5.08-2P-BK-S, J321 B04B-XASK-1, Q1 2N7002, Q2 2N7002, Q3 2N7002, Q4 2N7002, U1 DMP6023LE-13, U2 DMP6023LE-13, U3 DMP6023LE-13, U4 DMP6023LE-13

Commit message: gerber
Other:
- moved on the sheet: R18, R19, R20, R3

Commit message: 14.1.15 with PMOS fixed
Parts:
- removed U1, U2, U3, U4: DMP6023LE-13, PCB_Library:SOT230P700X185-4N, symbol PCB_Library:BSS308PEH6327XTSA1
- added Q10, Q5, Q6, Q7, Q8, Q9: DMP6023LE-PMOS, PCB_Library:SOT-223 DMP6023LE, symbol PCB_Library:DMP6023LE-PMOS
Connections:
- net at D10.1 (K), D11.1 (K), D13.1 (K)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: now also Q10.3 (S), Q5.3 (S), Q6.3 (S), Q8.3 (S)
- net at D1.2 (A), D16.1 (K), D309.1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: now also Q5.2 (D)
- net at D12.1 (K), D13.2 (A), D3.2 (A)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: now also Q10.2 (D)
- net at D10.2 (A), D15.1 (K), D2.2 (A)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: now also Q6.2 (D)
- net at R1.1, R17.2: now also Q5.1 (G)
- net at R18.1, R6.1: now also Q8.1 (G)
- net at D11.2 (A), D14.1 (K), D302.1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: now also Q8.2 (D)
- net at R20.1, R3.1: now also Q6.1 (G)
- net at R19.1, R7.1: now also Q10.1 (G)
