File: 14.1.5 - PMOS - PLC Connector Combined/12.1.1.a.kicad_sch (KiCad schematic)
At the start: 30 parts, among them J201 Conn_01x01_PAD, J202 Conn_01x01_PAD, J203 Conn_01x01_PAD, J204 Conn_01x01_PAD, J205 Conn_01x01_PAD, J206 Conn_01x01_PAD, J207 Conn_01x01_PAD, J208 Conn_01x01_PAD, J209 Conn_01x01_PAD, J210 Conn_01x01_PAD, J211 Conn_01x01_PAD, J212 Conn_01x01_PAD, J213 Conn_01x01_PAD, J214 Conn_01x01_PAD, J215 Conn_01x01_PAD, J216 Conn_01x01_PAD, J217 Conn_01x01_PAD, J218 Conn_01x01_PAD, J219 Conn_01x01_PAD, J220 Conn_01x01_PAD, J221 DB128L-5.08-2P-BK-S, J222 DB128L-5.08-2P-BK-S, J223 DB128L-5.08-2P-BK-S, J224 DB128L-5.08-2P-BK-S, J225 DB128L-5.08-2P-BK-S, J226 B04B-XASK-1

Commit message: 4.1.6
Parts:
- J226: footprint PCB_Library:CONN_B04B-XASK-1_JST -> PCB_Library:CONN_B04B-XASK-1-A_JST; LCSC C264994 -> C491709
Changed lines of the file:
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@@
       (effects (font (size 1.524 1.524)))
     )
-    (property "Footprint" "PCB_Library:CONN_B04B-XASK-1_JST" (at 220.98 95.25 0)
+    (property "Footprint" "PCB_Library:CONN_B04B-XASK-1-A_JST" (at 220.98 95.25 0)
       (effects (font (size 1.27 1.27) italic) hide)
     )
@@
       (effects (font (size 1.27 1.27) italic) hide)
     )
-    (property "LCSC" "C264994" (at 228.6 72.39 0)
+    (property "LCSC" "C491709" (at 228.6 72.39 0)
       (effects (font (size 1.27 1.27)))
     )
