File: 14.1.5 - PMOS - PLC Connector Combined/12.2.1.a.kicad_sch (KiCad schematic)
At the start: 69 parts, among them J301 Conn_01x01_PAD, J302 Conn_01x01_PAD, J303 Conn_01x01_PAD, J304 Conn_01x01_PAD, J305 Conn_01x01_PAD, J306 Conn_01x01_PAD, J307 Conn_01x01_PAD, J308 Conn_01x01_PAD, J309 Conn_01x01_PAD, J310 Conn_01x01_PAD, J311 Conn_01x01_PAD, J312 Conn_01x01_PAD, J313 Conn_01x01_PAD, J314 Conn_01x01_PAD, J315 Conn_01x01_PAD, J316 Conn_01x01_PAD, J317 DB128L-5.08-2P-BK-S, J318 DB128L-5.08-3P-BK-S, J319 DB128L-5.08-2P-BK-S, J320 DB128L-5.08-2P-BK-S, J321 B04B-XASK-1, Q1 2N7002, Q10 DMP6023LE-PMOS, Q2 2N7002, Q3 2N7002, Q4 2N7002, Q5 DMP6023LE-PMOS, Q6 DMP6023LE-PMOS, Q8 DMP6023LE-PMOS

Commit message: 4.1.6
Parts:
- J321: footprint PCB_Library:CONN_B04B-XASK-1_JST -> PCB_Library:CONN_B04B-XASK-1-A_JST; LCSC C264994 -> C491709
Changed lines of the file:
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@@
       (effects (font (size 1.524 1.524)) (justify left))
     )
-    (property "Footprint" "PCB_Library:CONN_B04B-XASK-1_JST" (at 264.16 138.43 0)
+    (property "Footprint" "PCB_Library:CONN_B04B-XASK-1-A_JST" (at 264.16 138.43 0)
       (effects (font (size 1.27 1.27) italic) hide)
     )
@@
       (effects (font (size 1.27 1.27) italic) hide)
     )
-    (property "LCSC" "C264994" (at 275.59 130.81 0)
+    (property "LCSC" "C491709" (at 275.59 130.81 0)
       (effects (font (size 1.27 1.27)) (justify left))
     )
