File: 14.1.5 - PMOS - PLC Connector Combined/14.1.5 - PMOS - PLC Connector Combined.kicad_pcb (KiCad board)
At the start: 2 copper layers, 61.5 x 67.8 mm, 110 parts, among them J201 Conn_01x01_PAD, J202 Conn_01x01_PAD, J203 Conn_01x01_PAD, J204 Conn_01x01_PAD, J205 Conn_01x01_PAD, J206 Conn_01x01_PAD, J207 Conn_01x01_PAD, J208 Conn_01x01_PAD, J209 Conn_01x01_PAD, J210 Conn_01x01_PAD, J211 Conn_01x01_PAD, J212 Conn_01x01_PAD, J213 Conn_01x01_PAD, J214 Conn_01x01_PAD, J215 Conn_01x01_PAD, J216 Conn_01x01_PAD, J217 Conn_01x01_PAD, J218 Conn_01x01_PAD, J219 Conn_01x01_PAD, J220 Conn_01x01_PAD, J221 DB128L-5.08-2P-BK-S, J222 DB128L-5.08-2P-BK-S, J223 DB128L-5.08-2P-BK-S, J224 DB128L-5.08-2P-BK-S, J225 DB128L-5.08-2P-BK-S, J226 B04B-XASK-1, J301 Conn_01x01_PAD, J302 Conn_01x01_PAD, J303 Conn_01x01_PAD, J304 Conn_01x01_PAD, J305 Conn_01x01_PAD, J306 Conn_01x01_PAD, J307 Conn_01x01_PAD, J308 Conn_01x01_PAD, J309 Conn_01x01_PAD, J310 Conn_01x01_PAD, J311 Conn_01x01_PAD, J312 Conn_01x01_PAD, J313 Conn_01x01_PAD, J314 Conn_01x01_PAD, J315 Conn_01x01_PAD, J316 Conn_01x01_PAD, J317 DB128L-5.08-2P-BK-S, J318 DB128L-5.08-3P-BK-S, J319 DB128L-5.08-2P-BK-S, J320 DB128L-5.08-2P-BK-S, J321 B04B-XASK-1, Q1 2N7002, Q10 DMP6023LE-PMOS, Q2 2N7002, Q3 2N7002, Q4 2N7002, Q5 DMP6023LE-PMOS, Q6 DMP6023LE-PMOS, Q8 DMP6023LE-PMOS

Commit message: 4.1.6
Parts:
- J226, J321: footprint PCB_Library:CONN_B04B-XASK-1_JST -> PCB_Library:CONN_B04B-XASK-1-A_JST
- moved J318 10.2 mm to (107.5, 79.2), turned to 90 degrees
- moved J224 5.08 mm to (92.6, 113.0), turned to -90 degrees
- moved J221 5.08 mm to (92.6, 102.8), turned to -90 degrees
- moved J222 5.08 mm to (92.6, 92.7), turned to -90 degrees
- moved J223 5.08 mm to (92.6, 72.3), turned to -90 degrees
- moved J225 5.08 mm to (92.6, 82.5), turned to -90 degrees
- moved J317 5.08 mm to (107.5, 94.1), turned to 90 degrees
- moved J319 5.08 mm to (107.5, 124.5), turned to 90 degrees
- moved J320 5.08 mm to (107.5, 109.1), turned to 90 degrees
