File: 14.1.7 - PMOS - PLC Connector Combined/12.1.1.a.kicad_sch (KiCad schematic)
At the start: 30 parts, among them J201 Conn_01x01_PAD, J202 Conn_01x01_PAD, J203 Conn_01x01_PAD, J204 Conn_01x01_PAD, J205 Conn_01x01_PAD, J206 Conn_01x01_PAD, J207 Conn_01x01_PAD, J208 Conn_01x01_PAD, J209 Conn_01x01_PAD, J210 Conn_01x01_PAD, J211 Conn_01x01_PAD, J212 Conn_01x01_PAD, J213 Conn_01x01_PAD, J214 Conn_01x01_PAD, J215 Conn_01x01_PAD, J216 Conn_01x01_PAD, J217 Conn_01x01_PAD, J218 Conn_01x01_PAD, J219 Conn_01x01_PAD, J220 Conn_01x01_PAD, J221 DB128L-5.08-2P-BK-S, J222 DB128L-5.08-2P-BK-S, J223 DB128L-5.08-2P-BK-S, J224 DB128L-5.08-2P-BK-S, J225 DB128L-5.08-2P-BK-S, J226 B04B-XASK-1

Commit message: updated 14.1.7
Parts:
- added D201, D202, D203, D204: LED WHITE, LED_SMD:LED_0603_1608Metric, symbol Device:LED
- added R205, R206, R207, R208: 4.7k, Resistor_SMD:R_0603_1608Metric, symbol Device:R
Connections:
- net M: now also R205.1, R206.1, R207.1, R208.1
- net at J205.1 (Pin_1), J215.1 (Pin_1), J222.1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: now also D203.2 (A)
- net at J206.1 (Pin_1), J216.1 (Pin_1), J222.2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: now also D204.2 (A)
- net at J203.1 (Pin_1), J213.1 (Pin_1), J221.1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: now also D201.2 (A)
- net at J204.1 (Pin_1), J214.1 (Pin_1), J221.2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: now also D202.2 (A)
- new net: D204.1 (K), R208.2
- new net: D202.1 (K), R206.2
- new net: D201.1 (K), R205.2
- new net: D203.1 (K), R207.2
Other:
- moved on the sheet: J224, R201, R202
