File: 14.1.7 - PMOS - PLC Connector Combined/14.1.7 - PMOS - PLC Connector Combined.kicad_pcb (KiCad board)
At the start: 2 copper layers, 61.5 x 67.8 mm, 118 parts, among them J201 Conn_01x01_PAD, J202 Conn_01x01_PAD, J203 Conn_01x01_PAD, J204 Conn_01x01_PAD, J205 Conn_01x01_PAD, J206 Conn_01x01_PAD, J207 Conn_01x01_PAD, J208 Conn_01x01_PAD, J209 Conn_01x01_PAD, J210 Conn_01x01_PAD, J211 Conn_01x01_PAD, J212 Conn_01x01_PAD, J213 Conn_01x01_PAD, J214 Conn_01x01_PAD, J215 Conn_01x01_PAD, J216 Conn_01x01_PAD, J217 Conn_01x01_PAD, J218 Conn_01x01_PAD, J219 Conn_01x01_PAD, J220 Conn_01x01_PAD, J221 DB128L-5.08-2P-BK-S, J222 DB128L-5.08-2P-BK-S, J223 DB128L-5.08-2P-BK-S, J224 DB128L-5.08-2P-BK-S, J225 DB128L-5.08-2P-BK-S, J226 B04B-XASK-1, J301 Conn_01x01_PAD, J302 Conn_01x01_PAD, J303 Conn_01x01_PAD, J304 Conn_01x01_PAD, J305 Conn_01x01_PAD, J306 Conn_01x01_PAD, J307 Conn_01x01_PAD, J308 Conn_01x01_PAD, J309 Conn_01x01_PAD, J310 Conn_01x01_PAD, J311 Conn_01x01_PAD, J312 Conn_01x01_PAD, J313 Conn_01x01_PAD, J314 Conn_01x01_PAD, J315 Conn_01x01_PAD, J316 Conn_01x01_PAD, J317 DB128L-5.08-2P-BK-S, J318 DB128L-5.08-3P-BK-S, J319 DB128L-5.08-2P-BK-S, J320 DB128L-5.08-2P-BK-S, J321 B04B-XASK-1, J322 Conn_01x01, J323 Conn_01x01, J324 Conn_01x01, J325 Conn_01x01, Q1 2N7002, Q10 DMP6023LE-PMOS, Q2 2N7002, Q3 2N7002, Q4 2N7002, Q5 DMP6023LE-PMOS, Q6 DMP6023LE-PMOS, Q8 DMP6023LE-PMOS

Commit message: updated 14.1.7
Parts:
- added D201: LED WHITE, LED_SMD:LED_0603_1608Metric, F.Cu at (84.2, 107.8)
- added D202: LED WHITE, LED_SMD:LED_0603_1608Metric, F.Cu at (84.4, 102.8)
- added D203: LED WHITE, LED_SMD:LED_0603_1608Metric, F.Cu at (84.2, 97.6)
- added D204: LED WHITE, LED_SMD:LED_0603_1608Metric, F.Cu at (84.2, 92.6)
- added R205: 4.7k, Resistor_SMD:R_0603_1608Metric, F.Cu at (86.0, 107.0)
- added R206: 4.7k, Resistor_SMD:R_0603_1608Metric, F.Cu at (86.0, 103.0)
- added R207: 4.7k, Resistor_SMD:R_0603_1608Metric, F.Cu at (85.8, 97.6)
- added R208: 4.7k, Resistor_SMD:R_0603_1608Metric, F.Cu at (86.0, 93.4)
- F1, F2, F3, F4: value Fuse_Small 3A -> Fuse_Small 5A
- moved R203 0.60 mm to (86.6, 89.0)
- moved R204 0.60 mm to (86.6, 83.8)
Routing:
- net Net-(D201-A): track 68.3 -> 54.8 mm, vias 4 -> 2
- net Net-(D204-A): track 82.2 -> 69.5 mm, vias 3 -> 1
- net GNDPWR: track 238.3 -> 249.8 mm, vias 48 -> 51
- net Net-(D203-A): track 77.3 -> 69.0 mm, vias 5 -> 3
- net M: track 107.8 -> 114.8 mm
- net Net-(D10-K): track 155.2 -> 152.7 mm
- net Net-(D204-K): track 0.00 -> 2.14 mm
- net Net-(D201-K): track 0.00 -> 2.12 mm
- net Net-(D202-K): track 0.00 -> 1.68 mm
- net Net-(D203-K): track 0.00 -> 1.62 mm
- net Net-(Q5-G): track 23.0 -> 24.1 mm
- net Net-(D202-A): track 57.4 -> 56.7 mm, vias 3 -> 1

Commit message: updated 14.1.7
Other:
- board text added: "A1"
- board text added: "A2"
- board text added: "A3"
- board text added: "A4"
Changed lines of the file:
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@@
     (effects (font (size 1.8288 1.8288) (thickness 0.4572) bold) (justify bottom mirror))
   )
-  (gr_text "5" (at 82.673 102.927 90) (layer "F.SilkS")
-    (effects (font (size 1.8288 1.8288) (thickness 0.4572) bold) (justify bottom))
-  )
-  (gr_text "8" (at 82.673 117.913 90) (layer "F.SilkS")
+  (gr_text "5" (at 82.2 102.927 90) (layer "F.SilkS")
+    (effects (font (size 1.8288 1.8288) (thickness 0.4572) bold) (justify bottom))
+  )
+  (gr_text "8" (at 82.2 117.913 90) (layer "F.SilkS")
     (effects (font (size 1.8288 1.8288) (thickness 0.4572) bold) (justify bottom))
   )
@@
     (effects (font (size 1.8288 1.8288) (thickness 0.4572) bold) (justify bottom))
   )
-  (gr_text "L" (at 83 72 90) (layer "F.SilkS")
-    (effects (font (size 1.8288 1.8288) (thickness 0.4572) bold) (justify bottom))
-  )
-  (gr_text "4" (at 82.927 97.593 90) (layer "F.SilkS")
+  (gr_text "L" (at 82.2 72 90) (layer "F.SilkS")
+    (effects (font (size 1.8288 1.8288) (thickness 0.4572) bold) (justify bottom))
+  )
+  (gr_text "4" (at 82.2 97.593 90) (layer "F.SilkS")
+    (effects (font (size 1.8288 1.8288) (thickness 0.4572) bold) (justify bottom))
+  )
+  (gr_text "A1" (at 85.2 112.6 90) (layer "F.SilkS")
     (effects (font (size 1.8288 1.8288) (thickness 0.4572) bold) (justify bottom))
   )
@@
     (effects (font (size 1.8288 1.8288) (thickness 0.4572) bold) (justify bottom))
   )
-  (gr_text "M" (at 82.8 77.4 90) (layer "F.SilkS")
-    (effects (font (size 1.8288 1.8288) (thickness 0.4572) bold) (justify bottom))
-  )
-  (gr_text "475R" (at 84.8 87.4 90) (layer "F.SilkS")
-    (effects (font (size 0.889 0.889) (thickness 0.1778) bold) (justify bottom))
-  )
-  (gr_text "3" (at 82.8 92.6 90) (layer "F.SilkS")
+  (gr_text "M" (at 82.2 77.4 90) (layer "F.SilkS")
+    (effects (font (size 1.8288 1.8288) (thickness 0.4572) bold) (justify bottom))
+  )
+  (gr_text "A2" (at 85.2 118 90) (layer "F.SilkS")
+    (effects (font (size 1.8288 1.8288) (thickness 0.4572) bold) (justify bottom))
+  )
+  (gr_text "A3\n" (at 85 82.4 90) (layer "F.SilkS")
+    (effects (font (size 1.8288 1.8288) (thickness 0.4572) bold) (justify bottom))
+  )
+  (gr_text "3" (at 82.2 92.6 90) (layer "F.SilkS")
     (effects (font (size 1.8288 1.8288) (thickness 0.4572) bold) (justify bottom))
   )
@@
     (effects (font (size 1.016 1.016) (thickness 0.254) bold) (justify left bottom))
   )
-  (gr_text "6" (at 82.546 108.007 90) (layer "F.SilkS")
+  (gr_text "6" (at 82.2 108.007 90) (layer "F.SilkS")
     (effects (font (size 1.8288 1.8288) (thickness 0.4572) bold) (justify bottom))
   )
@@
     (effects (font (size 1.016 1.016) (thickness 0.254) bold) (justify left bottom))
   )
-  (gr_text "475R" (at 84.8 82.4 90) (layer "F.SilkS")
+  (gr_text "475R" (at 87 79.4 90) (layer "F.SilkS")
     (effects (font (size 0.889 0.889) (thickness 0.1778) bold) (justify bottom))
   )
@@
     (effects (font (size 1.016 1.016) (thickness 0.254) bold) (justify left bottom))
   )
-  (gr_text "2" (at 82.673 87.306 90) (layer "F.SilkS")
-    (effects (font (size 1.8288 1.8288) (thickness 0.4572) bold) (justify bottom))
-  )
-  (gr_text "360R" (at 84.8 118.2 90) (layer "F.SilkS")
+  (gr_text "2" (at 82.2 87.306 90) (layer "F.SilkS")
+    (effects (font (size 1.8288 1.8288) (thickness 0.4572) bold) (justify bottom))
+  )
+  (gr_text "360R" (at 87 120.6 90) (layer "F.SilkS")
     (effects (font (size 0.889 0.889) (thickness 0.1778) bold) (justify bottom))
   )
@@
     (effects (font (size 1.8288 1.8288) (thickness 0.4572) bold) (justify bottom))
   )
+  (gr_text "A4" (at 84.8 87.4 90) (layer "F.SilkS")
+    (effects (font (size 1.8288 1.8288) (thickness 0.4572) bold) (justify bottom))
+  )
   (gr_text "5" (at 100.04525 103.015224 90) (layer "F.SilkS")
     (effects (font (size 1.8288 1.8288) (thickness 0.4572) bold) (justify bottom))
@@
     (effects (font (size 1.8288 1.8288) (thickness 0.4572) bold) (justify bottom))
   )
-  (gr_text "7" (at 82.673 113.087 90) (layer "F.SilkS")
+  (gr_text "7" (at 82.2 113.087 90) (layer "F.SilkS")
     (effects (font (size 1.8288 1.8288) (thickness 0.4572) bold) (justify bottom))
   )
@@
     (effects (font (size 1.8288 1.8288) (thickness 0.4572) bold) (justify bottom))
   )
-  (gr_text "1" (at 82.8 82.353 90) (layer "F.SilkS")
+  (gr_text "1" (at 82.2 82.353 90) (layer "F.SilkS")
     (effects (font (size 1.8288 1.8288) (thickness 0.4572) bold) (justify bottom))
   )
@@
     )
   )
-  (gr_text "360R" (at 84.8 112.8 90) (layer "F.SilkS")
-    (effects (font (size 0.889 0.889) (thickness 0.1778) bold) (justify bottom))
-  )
   (gr_text "L+" (at 100.04525 71.138224 90) (layer "F.SilkS")
